Commit message: updated hand urdf

File: togo_description/urdf/umbc_husky_full.urdf (robot description, URDF)
Before this commit: robot husky, 36 links, 35 joints
Joints:
- joint j2n6s300_joint_finger_1: origin xyz=0.00279 0.03126 -0.11467 rpy=-1.570796327 .649262481663582 1.35961148639407 -> xyz=0.00279 0.03126 -0.11467 rpy=-1.7047873384941834 0.6476144647144773 1.67317415161155
- joint top_plate_to_kinect2: origin xyz=-0.30 -0.08 0.57 rpy=-1.57079633 0 -1.57079633 -> xyz=-0.30 -0.1 0.57 rpy=-1.57079633 0 -1.57079633
- joint top_plate_to_right_arm: origin xyz=0.21 -0.197 0.315 rpy=0 0 0 -> xyz=0.22 -0.197 0.315 rpy=0 0 0
